Commit message: nowy urdf

File: Stepping/leg_left.urdf (robot description, URDF)
Before this commit: robot leg, 13 links, 12 joints
Links:
- removed link Part_2_3
- removed link Part_2_4
- removed link Segment1Lewy_v6_1
- removed link Segment1Lewy_v6_2
- removed link Segment3-4_v11_3
- removed link Segment3-4_v11_4
- removed link WJ-WK00-0018_45_10
- removed link WJ-WK00-0018_45_6
- removed link WJ-WK00-0018_45_7
- removed link WJ-WK00-0018_45_8
- removed link WJ-WK00-0018_45_9
Joints:
- removed joint Fastened_10
- removed joint Fastened_11
- removed joint Fastened_12
- removed joint Fastened_13
- removed joint Fastened_14
- removed joint Fastened_15
- removed joint Fastened_9
- removed joint Revolute_10
- removed joint Revolute_11
- removed joint Revolute_7
- removed joint Revolute_8
- removed joint Revolute_9

File: Stepping/leg_right.urdf (robot description, URDF)
Before this commit: robot leg, 13 links, 12 joints
Links:
- removed link Part_2_1
- removed link Part_2_2
- removed link Segment1Prawypierwszy_v7_1
- removed link Segment1Prawypierwszy_v7_2
- removed link Segment3-4_v11_1
- removed link Segment3-4_v11_2
- removed link WJ-WK00-0018_45_1
- removed link WJ-WK00-0018_45_2
- removed link WJ-WK00-0018_45_3
- removed link WJ-WK00-0018_45_4
- removed link WJ-WK00-0018_45_5
Joints:
- removed joint Fastened_1
- removed joint Fastened_2
- removed joint Fastened_3
- removed joint Fastened_4
- removed joint Fastened_5
- removed joint Fastened_6
- removed joint Revolute_1
- removed joint Revolute_2
- removed joint Revolute_3
- removed joint Revolute_4
- removed joint Revolute_5
- removed joint Revolute_6

File: beta.urdf (robot description, URDF)
Before this commit: robot quadruped, 29 links, 28 joints
Links:
- removed link Part_1_4_1
- removed link Segment1Lewy_v6_1
- removed link Segment1Lewy_v6_2
- removed link Segment1Prawypierwszy_v7_1
- removed link Segment1Prawypierwszy_v7_2
- removed link Segment3-4_v11_1
- removed link Segment3-4_v11_2
- removed link Segment3-4_v11_3
- removed link Segment3-4_v11_4
- removed link StopaLewa_v6_1
- removed link gacieOgarniete_v10_1
- added link Segment1Lewy_1, mass 0.015041115; collision mesh filename=meshes/Segment1Lewy_1.stl; visual mesh filename=meshes/Segment1Lewy_1.stl
- added link Segment1Lewy_2, mass 0.01; collision mesh filename=meshes/Segment1Lewy_2.stl; visual mesh filename=meshes/Segment1Lewy_2.stl
- added link Segment1Prawypierwszy_1, mass 0.015041115; collision mesh filename=meshes/Segment1Prawypierwszy_1.stl; visual mesh filename=meshes/Segment1Prawypierwszy_1.stl
- added link Segment1Prawypierwszy_2, mass 0.01; collision mesh filename=meshes/Segment1Prawypierwszy_2.stl; visual mesh filename=meshes/Segment1Prawypierwszy_2.stl
- added link Segment3-4_1, mass 0.043866671; collision mesh filename=meshes/Segment3-4_1.stl; visual mesh filename=meshes/Segment3-4_1.stl
- added link Segment3-4_2, mass 0.043866671; collision mesh filename=meshes/Segment3-4_2.stl; visual mesh filename=meshes/Segment3-4_2.stl
- added link Segment3-4_3, mass 0.043866671; collision mesh filename=meshes/Segment3-4_3.stl; visual mesh filename=meshes/Segment3-4_3.stl
- added link Segment3-4_4, mass 0.043866671; collision mesh filename=meshes/Segment3-4_4.stl; visual mesh filename=meshes/Segment3-4_4.stl
- added link StopaLewa_1, mass 0.036762237; collision mesh filename=meshes/StopaLewa_1.stl; visual mesh filename=meshes/StopaLewa_1.stl
- added link StopaPrawa_1, mass 0.036762326; collision mesh filename=meshes/Part_1_4_1.stl; visual mesh filename=meshes/Part_1_4_1.stl
- added link gacieOgarniete_1, mass 0.09292403; collision mesh filename=meshes/gacieOgarniete_1.stl; visual mesh filename=meshes/gacieOgarniete_1.stl
- link GE_27_1: mass 0 -> 0.092117424
- link GE_27_2: mass 0 -> 0.092117424
- link GE_27_3: mass 0 -> 0.092117424
- link Mocowanie_1: mass 0 -> 0.041493277
- link Part_2_1: mass 0 -> 0.03284794
- link Part_2_2: mass 0 -> 0.025206947
- link Part_2_3: mass 0 -> 0.025206947
- link Part_2_4: mass 0 -> 0.03284794
- link WJ-WK00-0018_45_1: mass 0 -> 0.03108367
- link WJ-WK00-0018_45_10: mass 0 -> 0.03108367
- link WJ-WK00-0018_45_2: mass 0 -> 0.03108367
- link WJ-WK00-0018_45_3: mass 0 -> 0.03108367
- link WJ-WK00-0018_45_4: mass 0 -> 0.03108367
- link WJ-WK00-0018_45_5: mass 0 -> 0.03108367
- link WJ-WK00-0018_45_6: mass 0 -> 0.03108367
- link WJ-WK00-0018_45_7: mass 0 -> 0.03108367
- link WJ-WK00-0018_45_8: mass 0 -> 0.03108367
- link WJ-WK00-0018_45_9: mass 0 -> 0.03108367
Joints:
- removed joint Fastened_15
- removed joint Fastened_16
- removed joint Revolute_8
- added joint Revolute_13: type revolute, parent Part_2_4, child WJ-WK00-0018_45_10, origin xyz=-0.03619738 0.02454328 0.02353646 rpy=-1.5707963 -1.5707963 0, axis 0 0 -1, limit lower=-6.2831853 upper=6.2831853 effort=1 velocity=1
- added joint Revolute_14: type revolute, parent Mocowanie_1, child GE_27_3, origin xyz=-0.05384144 -0.31946563 0.017528324 rpy=0.039065686 0 0, axis 0 0 -1, limit lower=-6.2831853 upper=6.2831853 effort=1 velocity=1
- added joint Revolute_8_Fixed: type fixed, parent Segment1Prawypierwszy_2, child Segment1Prawypierwszy_1, origin xyz=0 0 -0.005 rpy=0 0 -1.5707963
- joint Fastened_1: child Part_1_4_1 -> StopaLewa_1; origin xyz=-0.027 6.9e-07 -0.00885 rpy=0 0 0 -> xyz=-6.9e-07 0.027 0.00885 rpy=3.1415927 0 -1.5707963
- joint Fastened_10: child WJ-WK00-0018_45_6 -> WJ-WK00-0018_45_7; origin xyz=-0.0156 -0.02700504 -0.013 rpy=-1.5707963 0 1.5707963 -> xyz=0.02329868 0.01585672 0.024 rpy=-1.5707963 0 0; parent Segment1Lewy_v6_2 -> Part_2_3
- joint Fastened_11: child Part_2_3 -> WJ-WK00-0018_45_8; origin xyz=0.02700002 -7e-07 -0.0401 rpy=3.1415927 0 0 -> xyz=0 -0.0863 0.0404 rpy=0 0 -1.5707963; parent WJ-WK00-0018_45_6 -> Segment3-4_3
- joint Fastened_12: child WJ-WK00-0018_45_7 -> WJ-WK00-0018_45_9; origin xyz=0.01535671 -0.02329869 -0.025 rpy=-1.5707963 0 -1.5707963 -> xyz=0 -0.0863 0.0404 rpy=0 0 -1.5707963; parent Part_2_3 -> Segment3-4_4
- joint Fastened_13: child WJ-WK00-0018_45_8 -> StopaPrawa_1; origin xyz=0.0863 0 -0.0399 rpy=3.1415927 0 0 -> xyz=-0.027 6.9e-07 -0.00435 rpy=3.1415927 0 -1.5707963; parent Segment3-4_v11_3 -> WJ-WK00-0018_45_10
- joint Fastened_14: child WJ-WK00-0018_45_9 -> gacieOgarniete_1; origin xyz=0 -0.0863 0.0399 rpy=0 0 -1.5707963 -> xyz=-0.01025 -0.029 0.0032 rpy=3.1415927 0 -1.5707963; parent Segment3-4_v11_4 -> GE_27_3
- joint Fastened_2: parent Segment3-4_v11_1 -> Segment3-4_1
- joint Fastened_3: parent Segment3-4_v11_2 -> Segment3-4_2
- joint Fastened_4: origin xyz=0.01535671 0.02329869 -0.024 rpy=1.5707963 0 1.5707963 -> xyz=0.02035672 0.02329868 -0.024 rpy=-1.5707963 0 1.5707963
- joint Fastened_5: origin xyz=-0.0201 -0.02700504 0.013 rpy=-1.5707963 0 -1.5707963 -> xyz=-0.0201 -0.02700504 -0.013 rpy=1.5707963 0 1.5707963; parent Segment1Prawypierwszy_v7_1 -> Segment1Lewy_1
- joint Fastened_6: child Segment1Prawypierwszy_v7_1 -> Segment1Lewy_1; origin xyz=0 0 0.005 rpy=0 0 3.1415927 -> xyz=0 0 0.005 rpy=3.1415927 0 3.1415927; parent Segment1Prawypierwszy_v7_2 -> Segment1Lewy_2
- joint Fastened_7: origin xyz=0.00375 0.051 -0.00080765 rpy=0 0 0 -> xyz=0.00375 -0.051 -0.00080765 rpy=0 0 0; parent gacieOgarniete_v10_1 -> gacieOgarniete_1
- joint Fastened_8: origin xyz=0.00375 -0.051 -0.00080765 rpy=0 0 0 -> xyz=0.00375 0.0305 -0.00080765 rpy=0 0 0; parent gacieOgarniete_v10_1 -> gacieOgarniete_1
- joint Fastened_9: child Segment1Lewy_v6_2 -> WJ-WK00-0018_45_6; origin xyz=0 0 -0.003 rpy=0 0 0 -> xyz=-0.0156 0.02700504 -0.013 rpy=1.5707963 0 -1.5707963; parent Segment1Lewy_v6_1 -> Segment1Prawypierwszy_1
- joint Revolute_1: origin xyz=0.03619738 0.02353646 -0.02454329 rpy=-1.5707963 1.5707963 0 -> xyz=-0.03619738 -0.02454328 0.02546354 rpy=-1.5707963 0 0
- joint Revolute_10: child Part_2_4 -> Segment3-4_3; parent WJ-WK00-0018_45_9 -> WJ-WK00-0018_45_7
- joint Revolute_11: child WJ-WK00-0018_45_10 -> Segment3-4_4; origin xyz=0.02353646 -0.03619738 0.02445671 rpy=3.1415927 -1.5707963 0 -> xyz=0.027 -6.9e-07 0.00885 rpy=3.1415927 0 -1.5707963; parent Part_2_4 -> WJ-WK00-0018_45_8
- joint Revolute_12: child GE_27_3 -> Part_2_4; origin xyz=-0.085284089 -0.31119158 0.0032971737 rpy=-2.8999145 -1.1132852 3.1415926 -> xyz=0.027 -6.9e-07 0.00885 rpy=3.1415927 0 3.1415927; parent Mocowanie_1 -> WJ-WK00-0018_45_9
- joint Revolute_2: limit lower=4.5553093 upper=7.993608 effort=1 velocity=1 -> lower=-6.2831853 upper=6.2831853 effort=1 velocity=1; origin xyz=-6.9e-07 0.027 -0.00385 rpy=3.1415927 0 1.5707963 -> xyz=-6.9e-07 0.027 -0.00435 rpy=0 0 -1.5707963
- joint Revolute_3: child Segment3-4_v11_1 -> Segment3-4_1; limit lower=4.5553093 upper=7.993608 effort=1 velocity=1 -> lower=-6.2831853 upper=6.2831853 effort=1 velocity=1; origin xyz=-6.9e-07 0.027 -0.00385 rpy=3.1415927 0 1.5707963 -> xyz=-6.9e-07 0.027 -0.00435 rpy=3.1415927 0 1.5707963
- joint Revolute_4: child Segment3-4_v11_2 -> Segment3-4_2; origin xyz=0.027 -6.9e-07 0.00885 rpy=0 0 0 -> xyz=0.027 6.9e-07 -0.00435 rpy=3.1415927 0 0
- joint Revolute_5: origin xyz=-0.027 -6.9e-07 0.0446 rpy=0 0 3.1415927 -> xyz=0.027 6.9e-07 -0.00435 rpy=3.1415927 0 0
- joint Revolute_6: child Segment1Prawypierwszy_v7_2 -> Segment1Lewy_2
- joint Revolute_7: child Segment1Lewy_v6_1 -> Segment1Prawypierwszy_2; origin xyz=-0.03275 -0.01025 -0.0352 rpy=0 0 3.1415927 -> xyz=-0.03275 0.01025 -0.035 rpy=0 0 -1.5707963
- joint Revolute_9: child Segment3-4_v11_4 -> Part_2_3; origin xyz=0.027 -6.9e-07 0.00885 rpy=3.1415927 0 -1.5707963 -> xyz=0.027 -6.9e-07 -0.0401 rpy=0 0 -1.5707963; parent WJ-WK00-0018_45_8 -> WJ-WK00-0018_45_6

Commit message: nogi wygenerowane dla najnowszego urdf

File: Stepping/leg_left.urdf (robot description, URDF)
Before this commit: robot leg, 2 links, 0 joints
Links:
- removed link StopaLewa_v6_1
- added link GE_27_1
- added link Part_2_1
- added link Part_2_2
- added link Segment1Lewy_1
- added link Segment1Lewy_2
- added link Segment3-4_1
- added link Segment3-4_2
- added link StopaLewa_1
- added link WJ-WK00-0018_45_1
- added link WJ-WK00-0018_45_2
- added link WJ-WK00-0018_45_3
- added link WJ-WK00-0018_45_4
- added link WJ-WK00-0018_45_5
- added link gacieOgarniete_1
Joints:
- added joint Fastened_1: type fixed, parent WJ-WK00-0018_45_1, child StopaLewa_1, origin xyz=-6.9e-07 0.027 0.00885 rpy=3.1415927 0 -1.5707963
- added joint Fastened_2: type fixed, parent Segment3-4_1, child WJ-WK00-0018_45_2, origin xyz=0.0863 0 -0.0449 rpy=0 0 -1.5707963
- added joint Fastened_3: type fixed, parent Segment3-4_2, child WJ-WK00-0018_45_3, origin xyz=0.0863 0 -0.0449 rpy=0 0 -1.5707963
- added joint Fastened_4: type fixed, parent Part_2_2, child WJ-WK00-0018_45_4, origin xyz=0.02035672 0.02329868 -0.024 rpy=-1.5707963 0 1.5707963
- added joint Fastened_5: type fixed, parent Segment1Lewy_1, child WJ-WK00-0018_45_5, origin xyz=-0.0201 -0.02700504 -0.013 rpy=1.5707963 0 1.5707963
- added joint Fastened_6: type fixed, parent Segment1Lewy_2, child Segment1Lewy_1, origin xyz=0 0 0.005 rpy=3.1415927 0 3.1415927
- added joint Fastened_7: type fixed, parent gacieOgarniete_1, child GE_27_1, origin xyz=0.00375 -0.051 -0.00080765 rpy=0 0 0
- added joint Fastened_8: type fixed, parent gacieOgarniete_1, child GE_27_2, origin xyz=0.00375 0.0305 -0.00080765 rpy=0 0 0
- added joint Revolute_1: type revolute, parent Part_2_1, child WJ-WK00-0018_45_1, origin xyz=-0.03619738 -0.02454328 0.02546354 rpy=-1.5707963 0 0, axis 0 0 -1, limit lower=-3.1415926535 upper=3.1415926535 effort=1000 velocity=1000
- added joint Revolute_2: type revolute, parent WJ-WK00-0018_45_2, child Part_2_1, origin xyz=-6.9e-07 0.027 -0.00435 rpy=0 0 -1.5707963, axis 0 0 -1, limit lower=-3.1415926535 upper=3.1415926535 effort=1000 velocity=1000
- added joint Revolute_3: type revolute, parent WJ-WK00-0018_45_3, child Segment3-4_1, origin xyz=-6.9e-07 0.027 -0.00435 rpy=3.1415927 0 1.5707963, axis 0 0 -1, limit lower=-3.1415926535 upper=3.1415926535 effort=1000 velocity=1000
- added joint Revolute_4: type revolute, parent WJ-WK00-0018_45_4, child Segment3-4_2, origin xyz=0.027 6.9e-07 -0.00435 rpy=3.1415927 0 0, axis 0 0 -1, limit lower=-3.1415926535 upper=3.1415926535 effort=1000 velocity=1000
- added joint Revolute_5: type revolute, parent WJ-WK00-0018_45_5, child Part_2_2, origin xyz=0.027 6.9e-07 -0.00435 rpy=3.1415927 0 0, axis 0 0 -1, limit lower=-3.1415926535 upper=3.1415926535 effort=1000 velocity=1000
- added joint Revolute_6: type revolute, parent GE_27_1, child Segment1Lewy_2, origin xyz=-0.03275 -0.01025 -0.0352 rpy=3.1415927 0 0, axis 0 0 -1, limit lower=-3.1415926535 upper=3.1415926535 effort=1000 velocity=1000

File: Stepping/leg_right.urdf (robot description, URDF)
Before this commit: robot leg, 2 links, 0 joints
Links:
- removed link Part_1_4_1
- added link GE_27_2
- added link Part_2_3
- added link Part_2_4
- added link Segment1Prawypierwszy_1
- added link Segment1Prawypierwszy_2
- added link Segment3-4_3
- added link Segment3-4_4
- added link StopaPrawa_1
- added link WJ-WK00-0018_45_10
- added link WJ-WK00-0018_45_6
- added link WJ-WK00-0018_45_7
- added link WJ-WK00-0018_45_8
- added link WJ-WK00-0018_45_9
- added link gacieOgarniete_1
Joints:
- added joint Fastened_10: type fixed, parent Part_2_3, child WJ-WK00-0018_45_7, origin xyz=0.02329868 0.01585672 0.024 rpy=-1.5707963 0 0
- added joint Fastened_11: type fixed, parent Segment3-4_3, child WJ-WK00-0018_45_8, origin xyz=0 -0.0863 0.0404 rpy=0 0 -1.5707963
- added joint Fastened_12: type fixed, parent Segment3-4_4, child WJ-WK00-0018_45_9, origin xyz=0 -0.0863 0.0404 rpy=0 0 -1.5707963
- added joint Fastened_13: type fixed, parent WJ-WK00-0018_45_10, child StopaPrawa_1, origin xyz=-0.027 6.9e-07 -0.00435 rpy=3.1415927 0 -1.5707963
- added joint Fastened_7: type fixed, parent gacieOgarniete_1, child GE_27_1, origin xyz=0.00375 -0.051 -0.00080765 rpy=0 0 0
- added joint Fastened_8: type fixed, parent gacieOgarniete_1, child GE_27_2, origin xyz=0.00375 0.0305 -0.00080765 rpy=0 0 0
- added joint Fastened_9: type fixed, parent Segment1Prawypierwszy_1, child WJ-WK00-0018_45_6, origin xyz=-0.0156 0.02700504 -0.013 rpy=1.5707963 0 -1.5707963
- added joint Revolute_10: type revolute, parent WJ-WK00-0018_45_7, child Segment3-4_3, origin xyz=0.027 -6.9e-07 0.00885 rpy=3.1415927 0 -1.5707963, axis 0 0 -1, limit lower=-3.1415926535 upper=3.1415926535 effort=1000 velocity=1000
- added joint Revolute_11: type revolute, parent WJ-WK00-0018_45_8, child Segment3-4_4, origin xyz=0.027 -6.9e-07 0.00885 rpy=3.1415927 0 -1.5707963, axis 0 0 -1, limit lower=-3.1415926535 upper=3.1415926535 effort=1000 velocity=1000
- added joint Revolute_12: type revolute, parent WJ-WK00-0018_45_9, child Part_2_4, origin xyz=0.027 -6.9e-07 0.00885 rpy=3.1415927 0 3.1415927, axis 0 0 -1, limit lower=-3.1415926535 upper=3.1415926535 effort=1000 velocity=1000
- added joint Revolute_13: type revolute, parent Part_2_4, child WJ-WK00-0018_45_10, origin xyz=-0.03619738 0.02454328 0.02353646 rpy=-1.5707963 -1.5707963 0, axis 0 0 -1, limit lower=-3.1415926535 upper=3.1415926535 effort=1000 velocity=1000
- added joint Revolute_7: type revolute, parent GE_27_2, child Segment1Prawypierwszy_2, origin xyz=-0.03275 0.01025 -0.035 rpy=0 0 -1.5707963, axis 0 0 -1, limit lower=-3.1415926535 upper=3.1415926535 effort=1000 velocity=1000
- added joint Revolute_8_Fixed: type fixed, parent Segment1Prawypierwszy_2, child Segment1Prawypierwszy_1, origin xyz=0 0 -0.005 rpy=0 0 -1.5707963
- added joint Revolute_9: type revolute, parent WJ-WK00-0018_45_6, child Part_2_3, origin xyz=0.027 -6.9e-07 -0.0401 rpy=0 0 -1.5707963, axis 0 0 -1, limit lower=-3.1415926535 upper=3.1415926535 effort=1000 velocity=1000

Commit message: nowy ik_solver, generuje torso rotator jako 7 joint prawej nogi

File: Stepping/leg_left.urdf (robot description, URDF)
Before this commit: robot leg_leg_left, 15 links, 14 joints
Links:
- removed link GE_27_2
- removed link gacieOgarniete_1
Joints:
- removed joint Fastened_7
- removed joint Fastened_8
- joint Revolute_1: limit lower=-3.1415926535 upper=3.1415926535 effort=1000 velocity=1000 -> lower=-6.2831853 upper=6.2831853 effort=1 velocity=1
- joint Revolute_2: limit lower=-3.1415926535 upper=3.1415926535 effort=1000 velocity=1000 -> lower=-6.2831853 upper=6.2831853 effort=1 velocity=1
- joint Revolute_3: limit lower=-3.1415926535 upper=3.1415926535 effort=1000 velocity=1000 -> lower=-6.2831853 upper=6.2831853 effort=1 velocity=1
- joint Revolute_4: limit lower=-3.1415926535 upper=3.1415926535 effort=1000 velocity=1000 -> lower=-6.2831853 upper=6.2831853 effort=1 velocity=1
- joint Revolute_5: limit lower=-3.1415926535 upper=3.1415926535 effort=1000 velocity=1000 -> lower=-6.2831853 upper=6.2831853 effort=1 velocity=1
- joint Revolute_6: limit lower=-3.1415926535 upper=3.1415926535 effort=1000 velocity=1000 -> lower=-6.2831853 upper=6.2831853 effort=1 velocity=1

File: Stepping/leg_right.urdf (robot description, URDF)
Before this commit: robot leg_leg_right, 15 links, 14 joints
Links:
- removed link GE_27_1
- removed link StopaPrawa_1
- removed link gacieOgarniete_1
- added link Part_1_4_1
Joints:
- removed joint Fastened_7
- removed joint Fastened_8
- removed joint Revolute_8_Fixed
- added joint Revolute_8: type revolute, parent Segment1Prawypierwszy_2, child Segment1Prawypierwszy_1, origin xyz=0 0 -0.005 rpy=0 0 -1.5707963, axis 0 0 -1, limit lower=-6.2831853 upper=6.2831853 effort=1 velocity=1
- joint Fastened_13: child StopaPrawa_1 -> Part_1_4_1
- joint Revolute_10: limit lower=-3.1415926535 upper=3.1415926535 effort=1000 velocity=1000 -> lower=-6.2831853 upper=6.2831853 effort=1 velocity=1
- joint Revolute_11: limit lower=-3.1415926535 upper=3.1415926535 effort=1000 velocity=1000 -> lower=-6.2831853 upper=6.2831853 effort=1 velocity=1
- joint Revolute_12: limit lower=-3.1415926535 upper=3.1415926535 effort=1000 velocity=1000 -> lower=-6.2831853 upper=6.2831853 effort=1 velocity=1
- joint Revolute_13: limit lower=-3.1415926535 upper=3.1415926535 effort=1000 velocity=1000 -> lower=-6.2831853 upper=6.2831853 effort=1 velocity=1
- joint Revolute_7: limit lower=-3.1415926535 upper=3.1415926535 effort=1000 velocity=1000 -> lower=-6.2831853 upper=6.2831853 effort=1 velocity=1
- joint Revolute_9: limit lower=-3.1415926535 upper=3.1415926535 effort=1000 velocity=1000 -> lower=-6.2831853 upper=6.2831853 effort=1 velocity=1
