Commit message: jeszcze nowszy urdf

File: beta.urdf (robot description, URDF)
Before this commit: robot humanoid_beta, 29 links, 28 joints
Links:
- removed link StopaPrawa_1
- added link Part_1_4_1, mass 0.036762326; collision mesh filename=meshes/Part_1_4_1.stl; visual mesh filename=meshes/Part_1_4_1.stl
- link Segment1Lewy_1: mass 0.015041115 -> 0
- link Segment1Lewy_2: mass 0.01 -> 0.00078950187
- link Segment1Prawypierwszy_2: mass 0.01 -> 0.00078950187
Joints:
- removed joint Revolute_8_Fixed
- added joint Revolute_8: type revolute, parent Segment1Prawypierwszy_2, child Segment1Prawypierwszy_1, origin xyz=0 0 -0.005 rpy=0 0 -1.5707963, axis 0 0 -1, limit lower=-6.2831853 upper=6.2831853 effort=1 velocity=1
- joint Fastened_13: child StopaPrawa_1 -> Part_1_4_1

Commit message: Ładnie chodzi w pybullecie, po prostu urdf jest chujowy

File: beta.urdf (robot description, URDF)
Before this commit: robot humanoid_beta, 29 links, 28 joints
Links:
- removed link Part_1_4_1
- added link StopaPrawa_1, mass 0.036762326; collision mesh filename=meshes/Part_1_4_1.stl; visual mesh filename=meshes/Part_1_4_1.stl
- link Segment1Lewy_1: mass 0 -> 0.015041115
- link Segment1Lewy_2: mass 0.00078950187 -> 0.01
- link Segment1Prawypierwszy_2: mass 0.00078950187 -> 0.01
Joints:
- removed joint Revolute_8
- added joint Revolute_8_Fixed: type fixed, parent Segment1Prawypierwszy_2, child Segment1Prawypierwszy_1, origin xyz=0 0 -0.005 rpy=0 0 -1.5707963
- joint Fastened_13: child Part_1_4_1 -> StopaPrawa_1

Commit message: jeszcze nowszy urdf i meshe

File: beta.urdf (robot description, URDF)
Before this commit: robot humanoid_beta, 29 links, 28 joints
Links:
- removed link Mocowanie_1
- removed link Part_2_1
- removed link Part_2_4
- removed link StopaPrawa_1
- removed link WJ-WK00-0018_45_1
- removed link WJ-WK00-0018_45_10
- removed link WJ-WK00-0018_45_2
- removed link WJ-WK00-0018_45_3
- removed link WJ-WK00-0018_45_4
- removed link WJ-WK00-0018_45_5
- removed link WJ-WK00-0018_45_6
- removed link WJ-WK00-0018_45_7
- removed link WJ-WK00-0018_45_8
- removed link WJ-WK00-0018_45_9
- added link Biodra_1, mass 0.041493277; collision mesh filename=meshes/Biodra_1.stl; visual mesh filename=meshes/Biodra_1.stl
- added link Part_1_4_1, mass 0.036762326; collision mesh filename=meshes/Part_1_4_1.stl; visual mesh filename=meshes/Part_1_4_1.stl
- added link kostkaLewa_1, mass 0.03284794; collision mesh filename=meshes/kostkaLewa_1.stl; visual mesh filename=meshes/kostkaLewa_1.stl
- added link kostkaLewa_4, mass 0.03284794; collision mesh filename=meshes/kostkaLewa_4.stl; visual mesh filename=meshes/kostkaLewa_4.stl
- added link servoST3025-1_1, mass 0.03108367; collision mesh filename=meshes/servoST3025-1_1.stl; visual mesh filename=meshes/servoST3025-1_1.stl
- added link servoST3025-1_10, mass 0.03108367; collision mesh filename=meshes/servoST3025-1_10.stl; visual mesh filename=meshes/servoST3025-1_10.stl
- added link servoST3025-1_2, mass 0.03108367; collision mesh filename=meshes/servoST3025-1_2.stl; visual mesh filename=meshes/servoST3025-1_2.stl
- added link servoST3025-1_3, mass 0.03108367; collision mesh filename=meshes/servoST3025-1_3.stl; visual mesh filename=meshes/servoST3025-1_3.stl
- added link servoST3025-1_4, mass 0.03108367; collision mesh filename=meshes/servoST3025-1_4.stl; visual mesh filename=meshes/servoST3025-1_4.stl
- added link servoST3025-1_5, mass 0.03108367; collision mesh filename=meshes/servoST3025-1_5.stl; visual mesh filename=meshes/servoST3025-1_5.stl
- added link servoST3025-1_6, mass 0.03108367; collision mesh filename=meshes/servoST3025-1_6.stl; visual mesh filename=meshes/servoST3025-1_6.stl
- added link servoST3025-1_7, mass 0.03108367; collision mesh filename=meshes/servoST3025-1_7.stl; visual mesh filename=meshes/servoST3025-1_7.stl
- added link servoST3025-1_8, mass 0.03108367; collision mesh filename=meshes/servoST3025-1_8.stl; visual mesh filename=meshes/servoST3025-1_8.stl
- added link servoST3025-1_9, mass 0.03108367; collision mesh filename=meshes/servoST3025-1_9.stl; visual mesh filename=meshes/servoST3025-1_9.stl
- link Segment1Lewy_1: mass 0.015041115 -> 0.015041122
- link Segment1Lewy_2: mass 0.01 -> 0.00078950187
- link Segment1Prawypierwszy_2: mass 0.01 -> 0.00078950187
Joints:
- removed joint Fastened_1
- removed joint Revolute_1
- removed joint Revolute_8_Fixed
- added joint Revolute_8: type revolute, parent Segment1Prawypierwszy_2, child Segment1Prawypierwszy_1, origin xyz=0 0 -0.005 rpy=0 0 -1.5707963, axis 0 0 -1, limit lower=-6.2831853 upper=6.2831853 effort=1 velocity=1
- added joint servoST3025-1_to_kostkaLewa: type revolute, parent kostkaLewa_1, child servoST3025-1_1, origin xyz=-0.03619738 -0.02454328 0.02546354 rpy=-1.5707963 0 0, axis 0 0 -1, limit lower=-6.2831853 upper=6.2831853 effort=1 velocity=1
- added joint stopaLewa_to_servoST3025-1: type fixed, parent servoST3025-1_1, child StopaLewa_1, origin xyz=-6.9e-07 0.027 0.00885 rpy=3.1415927 0 -1.5707963
- joint Fastened_10: child WJ-WK00-0018_45_7 -> servoST3025-1_7
- joint Fastened_11: child WJ-WK00-0018_45_8 -> servoST3025-1_8
- joint Fastened_12: child WJ-WK00-0018_45_9 -> servoST3025-1_9
- joint Fastened_13: child StopaPrawa_1 -> Part_1_4_1; parent WJ-WK00-0018_45_10 -> servoST3025-1_10
- joint Fastened_2: child WJ-WK00-0018_45_2 -> servoST3025-1_2
- joint Fastened_3: child WJ-WK00-0018_45_3 -> servoST3025-1_3
- joint Fastened_4: child WJ-WK00-0018_45_4 -> servoST3025-1_4
- joint Fastened_5: child WJ-WK00-0018_45_5 -> servoST3025-1_5
- joint Fastened_9: child WJ-WK00-0018_45_6 -> servoST3025-1_6
- joint Revolute_10: parent WJ-WK00-0018_45_7 -> servoST3025-1_7
- joint Revolute_11: parent WJ-WK00-0018_45_8 -> servoST3025-1_8
- joint Revolute_12: child Part_2_4 -> kostkaLewa_4; parent WJ-WK00-0018_45_9 -> servoST3025-1_9
- joint Revolute_13: child WJ-WK00-0018_45_10 -> servoST3025-1_10; parent Part_2_4 -> kostkaLewa_4
- joint Revolute_14: parent Mocowanie_1 -> Biodra_1
- joint Revolute_2: child Part_2_1 -> kostkaLewa_1; parent WJ-WK00-0018_45_2 -> servoST3025-1_2
- joint Revolute_3: parent WJ-WK00-0018_45_3 -> servoST3025-1_3
- joint Revolute_4: parent WJ-WK00-0018_45_4 -> servoST3025-1_4
- joint Revolute_5: parent WJ-WK00-0018_45_5 -> servoST3025-1_5
- joint Revolute_9: parent WJ-WK00-0018_45_6 -> servoST3025-1_6
